File: pcb-hat/pcb-hat.kicad_pcb (KiCad board)
At the start: 4 copper layers, 65 x 56.5 mm, 84 parts, among them Q1 Q_PMOS_GSD, Q2 Q_NPN, Q3 PJA3404A_R1_00001, Q4 Q_PMOS_GSD, Q5 Q_NPN, Q6 Q_PMOS_GSD, Q7 NMOS, U1 Headers, U2 HTD Servo, U3 INA219AxD, U4 INA180A1, U5 TL431DBZ, U6 AP63301WU-7, U8 LM3489, U9 Raspberry_Pi_Generic

Commit message: i lied and now im done editing for the day; things are shorting but at least the ratsnest is all gone
Parts:
- moved G*** 36.3 mm to (125.5, 107.9)
Routing:
- net +5V: track 176.0 -> 127.2 mm
- net GND: track 187.6 -> 220.5 mm, vias 8 -> 6
- net VCC: track 138.9 -> 107.9 mm
- net +3V3: track 56.2 -> 34.1 mm
- net /PI_SIGNAL: track 13.2 -> 33.4 mm, vias 0 -> 3
- net /SERVO_RP_LED: track 0.00 -> 2.93 mm
- net Net-(R11-Pad1): track 46.6 -> 47.5 mm
- removed copper zone on In2.Cu, net +BATT
- removed copper zone on In2.Cu, net VCC_LOAD
- removed copper zone on In2.Cu, net VDC
